File: Arduino Uno ISP Shield.sch (KiCad schematic (older format))
At the start: 25 parts, among them J1 CONN_POWER, J10 Conn_01x01_Female, J2 CONN_ANALOG_IN, J3 Conn_01x02_Male, J34 CONN_DIGITAL_8-13, J35 CONN_DIGITAL_0-7, J4 Conn_02x03_Odd_Even, J5 Conn_01x01_Female, J6 Conn_01x01_Female, J7 Conn_01x01_Female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

Commit message: Add fabrication data
Connections:
- no-connect marks 41 -> 40
Changed lines of the file:
@@
 NoConn ~ 6800 4200
 NoConn ~ 6800 4300
-NoConn ~ 5200 3900
 Text Notes 8200 1200 0    50   ~ 0
 STATUS LEDS
